File: Schematics/StitchReg.kicad_sch (KiCad schematic)
At the start: 10 parts, among them J1 Barrel_Jack, J2 DIN-6, K1 DIPxx-1Axx-11x, SW1 SW_Push, U1 MCP4131-xxxx-P

Commit message: fix schematics
Connections:
- net at K1.2: now also A1.17 (D2); no longer A1.3 (~{RESET})
- net at A1.10 (A1): no longer U1.1 (~{CS})
- net at A1.12 (A3): no longer U1.3 (SDI/SDO)
- net at A1.13 (SDA/A4): no longer U1.2 (SCK)
- net at A1.20 (D5): now also J2.1
- net at A1.21 (D6): now also J2.5
- net at A1.23 (D8): now also BZ1.2 (-)
- net at A1.25 (D10): now also U1.1 (~{CS})
- net at A1.27 (D12): now also U1.3 (SDI/SDO)
- net at A1.28 (D13): now also U1.2 (SCK)
- net at A1.5 (+5V): no longer J2.1
- net at A1.6 (GND): no longer J2.5
- net at A1.8 (VIN): no longer BZ1.2 (-)
Other:
- moved on the sheet: BZ1
