File: Schematics/StitchReg-Teensy/StitchReg-Teensy.kicad_sch (KiCad schematic)
At the start: 16 parts, among them J1 SensorJack, J2 Barrel_Jack, Q1 PN2222A, SW1 SW_Run, SW2 SW_Mode, SW3 SW_Up, SW4 SW_Down, SW5 SW_Sub, SW6 SW_Cut, U1 Teensy4.0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

Commit message: fix power symbol
Connections:
- net VSS: no longer DS1.2 (VDD), J1.T, R5.1, U2.8 (V_{DD})
- new net +5V: DS1.2 (VDD), J1.T, R5.1, U2.8 (V_{DD})

Commit message: update schematics with info
Other:
- company: (none) -> Stitch The Planet
Changed lines of the file:
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@@
 	(generator "eeschema")
 	(generator_version "9.0")
-	(paper "A4")
+	(paper "USLetter")
 	(title_block
 		(title "Stitch Regulator")
+		(date "2025-09-25")
 		(rev "2")
+		(company "Stitch The Planet")
 	)
 	(junction
